Commit message: redesigned&&lidar+IMU

File: description/urdf/cart_org.urdf (robot description, URDF)
Before this commit: robot cartbot, 8 links, 7 joints
Links:
- removed link base_footprint
- removed link imu_link
- removed link lidar_link
Joints:
- removed joint base_footprint_joint
- removed joint imu_joint
- removed joint lidar_joint
- joint front_left_wheel_joint: origin xyz=0 0.13 0.0 rpy=0 0 0 -> xyz=0.15 0.18 0.0 rpy=0 0 0
- joint front_right_wheel_joint: origin xyz=0 -0.13 0.0 rpy=0 0 0 -> xyz=0.15 -0.18 0.0 rpy=0 0 0
- joint rear_left_caster_joint: origin xyz=0.24 0 0.0 rpy=0 0 0 -> xyz=-0.15 0.18 0.0 rpy=0 0 0
- joint rear_right_caster_joint: origin xyz=-0.24 0 0.0 rpy=0 0 0 -> xyz=-0.15 -0.18 0.0 rpy=0 0 0
